File: business_card.kicad_pcb (KiCad board)
At the start: 2 copper layers, 85.6 x 54 mm, 2 parts, among them U1 NT3H2111

Commit message: feat: update CTA to "CAREFUL. IT THINKS." and set ENIG copper finish
- Replace "TAP YOUR PHONE TO TALK TO MY AI" with "CAREFUL. IT THINKS."
- Larger 3.5mm bold text for impact
- Set copper finish to ENIG (gold) for transparent card aesthetic
- Set solder mask to transparent for clear substrate rendering

Co-Authored-By: Claude Opus 4.6 <noreply@anthropic.com>
Other:
- board text added: "CAREFUL. IT THINKS."
- board text removed: "TAP YOUR PHONE TO TALK TO MY AI"
Changed lines of the file:
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@@
 			(layer "F.Mask"
 				(type "Top Solder Mask")
+				(color "#00000000")
 				(thickness 0.01)
 			)
@@
 			(layer "B.Mask"
 				(type "Bottom Solder Mask")
+				(color "#00000000")
 				(thickness 0.01)
 			)
@@
 				(type "Bottom Silk Screen")
 			)
-			(copper_finish "None")
+			(copper_finish "ENIG")
 			(dielectric_constraints no)
 		)
@@
 		)
 	)
-	(gr_text "TAP YOUR PHONE TO TALK TO MY AI"
+	(gr_text "CAREFUL. IT THINKS."
 		(at 142.8 110 0)
 		(layer "B.SilkS")
 		(effects
 			(font
-				(size 2.2 2.2)
-				(thickness 0.3)
+				(size 3.5 3.5)
+				(thickness 0.45)
 				(bold yes)
 			)

Commit message: feat: embed real QR code for mattcoburn.ai/card on back silkscreen (THE-183)
Replace placeholder rectangle and "QR CODE" label with 332 filled
silkscreen modules encoding https://mattcoburn.ai/card (QR version 2,
error correction M, 25x25 matrix, 0.72mm module size). Mirrored
horizontally for correct back-side scanning. DRC clean.

Co-Authored-By: Claude Opus 4.6 <noreply@anthropic.com>
Other:
- board text removed: "QR CODE"
